Commit message: modify pkg cdpr_gazebo

File: src/cdpr_description/xacro/cdpr_gazebo.xacro (robot description, xacro)
@@ -7,8 +7,4 @@
     <mu1>0.2</mu1>
     <mu2>0.2</mu2>
-    <kp>10000000</kp>
-    <kd>1</kd>
-    <minDepth>0.01</minDepth>
-    <maxVel>100</maxVel>
     <material>Gazebo/Blue</material>
   </gazebo>
@@ -16,8 +12,4 @@
     <mu1>0.2</mu1>
     <mu2>0.2</mu2>
-    <kp>10000000</kp>
-    <kd>1</kd>
-    <minDepth>0.01</minDepth>
-    <maxVel>100</maxVel>
     <material>Gazebo/Blue</material>
   </gazebo>
@@ -25,8 +17,4 @@
     <mu1>0.2</mu1>
     <mu2>0.2</mu2>
-    <kp>10000000</kp>
-    <kd>1</kd>
-    <minDepth>0.01</minDepth>
-    <maxVel>100</maxVel>
     <material>Gazebo/Blue</material>
   </gazebo>
@@ -34,8 +22,4 @@
     <mu1>0.2</mu1>
     <mu2>0.2</mu2>
-    <kp>10000000</kp>
-    <kd>1</kd>
-    <minDepth>0.01</minDepth>
-    <maxVel>100</maxVel>
     <material>Gazebo/Blue</material>
   </gazebo>
@@ -43,8 +27,4 @@
     <mu1>5</mu1>
     <mu2>5</mu2>
-    <kp>10000000</kp>
-    <kd>1</kd>
-    <minDepth>0.01</minDepth>
-    <maxVel>100</maxVel>
     <material>Gazebo/Orange</material>
   </gazebo>
@@ -52,8 +32,4 @@
     <mu1>5</mu1>
     <mu2>5</mu2>
-    <kp>10000000</kp>
-    <kd>1</kd>
-    <minDepth>0.01</minDepth>
-    <maxVel>100</maxVel>
     <material>Gazebo/Orange</material>
   </gazebo>
@@ -61,8 +37,4 @@
     <mu1>5</mu1>
     <mu2>5</mu2>
-    <kp>10000000</kp>
-    <kd>1</kd>
-    <minDepth>0.01</minDepth>
-    <maxVel>100</maxVel>
     <material>Gazebo/Orange</material>
   </gazebo>
@@ -70,8 +42,4 @@
     <mu1>5</mu1>
     <mu2>5</mu2>
-    <kp>10000000</kp>
-    <kd>1</kd>
-    <minDepth>0.01</minDepth>
-    <maxVel>100</maxVel>
     <material>Gazebo/Orange</material>
   </gazebo>

File: src/cdpr_urdf/urdf/cdpr_urdf.urdf (robot description, URDF)
Before this commit: robot cdpr_urdf, 9 links, 8 joints
Joints:
- joint joint_roll_rb: axis 0 1 0 -> 0 -1 0
- joint joint_roll_rf: axis 0 1 0 -> 0 -1 0
- joint joint_steer_lb: axis 0 0 -1 -> 0 0 1
