Commit message: modify pkg to run with ros_control

File: src/cdpr_description/xacro/cdpr.xacro (robot description, xacro)
@@ -5,7 +5,8 @@
 <robot
   name="cdpr" xmlns:xacro="http://www.ros.org/wiki/xacro">
-  <!-- 导入机器人urdf文件，SW插件生成可能会有错，需先修改好 -->
+  <!-- import cdpr urdf file，which is automatically generated by solidworks plugin.  -->
+  <!-- some details might be wrong and need to be fixed after generation. -->
   <xacro:include filename="$(find cdpr_urdf)/urdf/cdpr_urdf.urdf"/>
-  <!-- 添加world连杆和fixed关节 -->
+  <!-- add link dummy and fixed joint to base link -->
   <link name="dummy"/>
   <joint name="dummy_joint" type="fixed">
@@ -13,4 +14,22 @@
     <child link="base_link" />
   </joint>
-  <xacro:include filename="$(find cdpr_description)/xacro/cdpr_gazebo.xacro"/>
+  <gazebo reference="base_link">
+    <material>Gazebo/Red</material>
+  </gazebo>
+  <!-- add the following so as to use ros_control in gazebo-->
+  <!-- ros_control plugin -->
+  <gazebo>
+    <plugin name="gazebo_ros_control" filename="libgazebo_ros_control.so">
+      <robotNamespace>/cdpr</robotNamespace>
+      <robotSimType>gazebo_ros_control/DefaultRobotHWSim</robotSimType>
+    </plugin>
+  </gazebo>
+  <!-- Add transmission elements to URDF -->
+  <xacro:arg name="load_chassis" default="true"/>
+  <xacro:arg name="load_anchor_module" default="true"/>
+  <xacro:arg name="load_cable_module" default="true"/>
+  <xacro:if value="$(arg load_chassis)">
+      <xacro:include filename="$(find cdpr_description)/xacro/chassis.xacro"/>
+      <xacro:chassis/>
+  </xacro:if>
 </robot>

File: src/cdpr_urdf/urdf/cdpr_urdf.urdf (robot description, URDF)
Before this commit: robot cdpr_urdf, 9 links, 8 joints
Joints:
- removed joint joint_roll_lb
- removed joint joint_roll_lf
- removed joint joint_roll_rb
- removed joint joint_roll_rf
- removed joint joint_steer_lb
- removed joint joint_steer_lf
- removed joint joint_steer_rb
- removed joint joint_steer_rf
